File: DAPLink/Probes/DAPule/DAPule-LPC11U35/DAPule-LPC11U35-v1.1.0/DAPule-LPC11U35-v1.1.0.brd (EAGLE design)
At the start: 49.3 x 25.9 mm, 41 parts, among them CON14 SWD-10/TC2050_SMD, CON9 USB_MICROB, IC1 USBLC6-2SC6, IC2 LD1117S33, IC3 LPC11U35FHI33/501, Q1 12MHz, SW1 SKRKAEE010, T1 BSS84

Commit message: More reorganistion
Parts:
- removed TP11, TP12: PTR1TP07R, blackbriar:TP07R
- added CON2: SWD-10/TC2050_SMD, mbed-HDK-Connector:FTSH-105-02
- added TP2, TP5: PTR1TP07R, blackbriar:TP07R
- TP1: value PTR1TP16R -> PTR1TP07R; device blackbriar:TP16R -> blackbriar:TP07R
- moved TP1 26.3 mm to (19.7, -4.95)
- moved CON14 6.73 mm to (43.9, 3.81)
- moved TP8 3.12 mm to (23.4, -3.17)
- moved TP13 2.56 mm to (21.5, -4.32)
- moved TP9 0.40 mm to (18.7, -5.84)
Connections:
- new net N$1: IC3.22, TP1.TP
- new net N$5: IC3.26, TP2.TP
- new net N$6: IC3.28, TP5.TP
- net +3.3V_IF: now also CON2.1
- net GND: now also CON2.9
- net IF_NRESET: now also CON2.10
- net IF_SWCLK: now also CON2.4; no longer TP12.TP
- net IF_SWDIO: now also CON2.2; no longer TP11.TP
- net V_ISENSE: no longer TP1.TP
Routing:
- net IF_NRESET: track 9.22 -> 43.3 mm, vias 0 -> 4
- net IF_SWCLK: track 3.32 -> 34.4 mm, vias 0 -> 2
- net IF_SWDIO: track 1.45 -> 28.3 mm, vias 0 -> 2
- net IF_GPIO: track 51.5 -> 30.8 mm, vias 1 -> 3
- net TGT_NRESET: track 47.2 -> 54.2 mm, vias 3 -> 2
- net TGT_SWDIO: track 27.6 -> 34.2 mm
- net TGT_SWCLK: track 38.5 -> 43.8 mm
- net N$6: track 0.00 -> 5.06 mm
- net +3.3V_IF: track 27.4 -> 30.7 mm, vias 8 -> 9
- net TGT_RX: track 27.6 -> 24.4 mm
- net TGT_TX: track 27.1 -> 30.2 mm
- net IF_SDA: track 31.2 -> 28.2 mm
- net GND: track 4.86 -> 7.71 mm
- net N$1: track 0.00 -> 2.57 mm
- net PIO0_14: track 4.81 -> 2.48 mm
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Other:
- board text added: "DAPule-LPC11U35 v1.1.0"
- board text added: "LPC11U35"
- board text added: "TARGET"
- board text removed: "DAPule-LPC11U35 v1.0.0"

Commit message: Refactor of repository
Parts:
- removed C15: 18pF, mbed-HDK:0603
- removed CON14: SWD-10/TC2050_SMD, mbed-HDK-Connector:FTSH-105-02
- removed R13: 470R, mbed-HDK:0603@1
- removed R18: 33R, mbed-HDK:0603@1
- added C2: 10uF, mbed-HDK:0603
- added CON3: SWD-10/TC2050_SMD, mbed-HDK-Connector:FTSH-105-02
- added R2: 470R, mbed-HDK:0603@1
- added R4: 0R@DNF, mbed-HDK:0402@1
- C1: value 10uF -> 100nF
- C6: value 100nF -> 18pF
- D1: device mbed-HDK:BAT60A -> mbed-HDK-Transistor:SOD323
- R1: value 0R@DNF -> 470R; device mbed-HDK:0402@1 -> mbed-HDK:0603@1
- R11: value 470R -> 33R
- moved R11 17.2 mm to (11.4, -2.03), turned to 0 degrees
- moved CON2 12.3 mm to (43.9, 3.43)
- moved C6 8.63 mm to (15.6, 6.60), turned to 90 degrees
- moved R1 7.44 mm to (22.4, -8.38), turned to 270 degrees
- moved C1 1.40 mm to (7.87, 2.79)
- renumbered C12 to C4, C16 to C7, C17 to C9, C18 to C8, C19 to C3, C20 to C5, CON9 to CON1, LED4 to LED3, LED5 to LED1, LED6 to LED2, R12 to R3, R15 to R6, R16 to R5, R17 to R10, R19 to R9, R20 to R7, R21 to R8
Connections:
- net +3.3V_IF: now also C2.1, CON3.1, R1.1, R2.1; no longer C6.1, CON2.1, R11.1, R13.1
- net GND: now also C2.2, CON2.3, CON2.5, CON3.9; no longer C15.2, CON14.3, CON14.5, CON14.9
- net IF_NRESET: now also CON3.10; no longer CON2.10
- net IF_SWCLK: now also CON3.4; no longer CON2.4
- net IF_SWDIO: now also CON3.2; no longer CON2.2
- net N$18: now also C6.1; no longer C15.1
- net N$2: now also R2.2; no longer R11.2
- net N$7: now also R1.2; no longer R13.2
- net TGT_NRESET: now also CON2.10; no longer CON14.10
- net TGT_RTS: now also R4.2; no longer R1.2
- net TGT_RX: now also CON2.8; no longer CON14.8
- net TGT_SWCLK: now also CON2.4, R4.1; no longer CON14.4, R1.1
- net TGT_SWDIO: now also CON2.2; no longer CON14.2
- net TGT_TX: now also CON2.7; no longer CON14.7
- net USB-D+: now also R11.1; no longer R18.1
- net USB_DP: now also R11.2; no longer R18.2
- net V_ISENSE: now also CON2.1; no longer CON14.1
Routing:
- net +3.3V_IF: track 30.7 -> 28.9 mm
- net TGT_NRESET: track 54.2 -> 55.1 mm
- net IF_GPIO: track 30.8 -> 30.1 mm, vias 3 -> 2
Other:
- board text removed: "DAPlink"
