File: DAPLink/Probes/DAPule/DAPule-LPC11U35/DAPule-LPC11U35-v1.1.0/DAPule-LPC11U35-v1.1.0.sch (EAGLE design)
At the start: 41 parts, among them CON14 SWD-10/TC2050_SMD, CON9 USB_MICROB, IC1 USBLC6-2SC6, IC2 LD1117S33, IC3 LPC11U35FHI33/501, Q1 12MHz, SW1 SKRKAEE010, T1 BSS84

Commit message: More reorganistion
Parts:
- removed TP11, TP12: PTR1TP07R, blackbriar:PTR1TP07R
- added CON2: SWD-10/TC2050_SMD, mbed-HDK-Connector:SWD-10/TC2050_SMD
- added TP2, TP5: PTR1TP07R, blackbriar:PTR1TP07R
- TP1: value PTR1TP16R -> PTR1TP07R; device blackbriar:PTR1TP16R -> blackbriar:PTR1TP07R
Connections:
- new net N$1: IC3.TMS/PIO0_12/AD1/CT32B1_CAP0, TP1.TP
- new net N$5: IC3.PIO0_16/AD5/CT32B1_MAT3/WAKEUP, TP2.TP
- new net N$6: IC3.PIO1_15/!DCD!/CT16B0_MAT2/SCK1, TP5.TP
- net +3.3V_IF: now also CON2.VCC
- net GND: now also CON2.GND@9
- net IF_NRESET: now also CON2.NRESET
- net IF_SWCLK: now also CON2.SWCLK; no longer TP12.TP
- net IF_SWDIO: now also CON2.SWDIO; no longer TP11.TP
- net V_ISENSE: no longer TP1.TP
Other:
- note removed: "R7 enables the button to be held dow non power up to put LPC11U35 into ISP mode. To disable this, remove R7, and fit R6 instead."
Changed lines of the file:
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@@
 <part name="TP8" library="blackbriar" deviceset="PTR1" device="TP07R"/>
 <part name="TP9" library="blackbriar" deviceset="PTR1" device="TP07R"/>
-<part name="TP11" library="blackbriar" deviceset="PTR1" device="TP07R"/>
-<part name="TP12" library="blackbriar" deviceset="PTR1" device="TP07R"/>
 <part name="TP13" library="blackbriar" deviceset="PTR1" device="TP07R"/>
 <part name="SW1" library="mbed-HDK-Switch" deviceset="SKRKAEE010" device=""/>
 <part name="C1" library="mbed-HDK" deviceset="C" device="0603" value="10uF"/>
 <part name="PWR1" library="mbed-HDK" deviceset="+3.3V_IF" device=""/>
-<part name="TP1" library="blackbriar" deviceset="PTR1" device="TP16R" value="PTR1TP16R"/>
 <part name="R1" library="mbed-HDK" deviceset="R" device="0402" value="0R@DNF"/>
+<part name="GND1" library="mbed-HDK" deviceset="GND" device=""/>
+<part name="PWR2" library="mbed-HDK" deviceset="+3.3V_IF" device=""/>
+<part name="CON2" library="mbed-HDK-Connector" deviceset="SWD-10/TC2050" device="_SMD"/>
+<part name="TP1" library="blackbriar" deviceset="PTR1" device="TP07R"/>
+<part name="TP2" library="blackbriar" deviceset="PTR1" device="TP07R"/>
+<part name="TP5" library="blackbriar" deviceset="PTR1" device="TP07R"/>
 </parts>
 <sheets>
@@
 <sheet>
 <plain>
-<text x="144.78" y="152.4" size="1.778" layer="97" font="vector" ratio="12">R7 enables the button to be held dow non power up to put LPC11U35 into ISP mode.
-To disable this, remove R7, and fit R6 instead.</text>
 <text x="7.62" y="175.26" size="1.778" layer="97" font="vector" ratio="12">Closing this jumper enables original
 firmware without flow control support
@@
 <instance part="TP8" gate="G$1" x="218.44" y="88.9" rot="R180"/>
 <instance part="TP9" gate="G$1" x="218.44" y="91.44" rot="R180"/>
-<instance part="TP11" gate="G$1" x="45.72" y="68.58"/>
-<instance part="TP12" gate="G$1" x="45.72" y="81.28"/>
 <instance part="TP13" gate="G$1" x="45.72" y="71.12"/>
 <instance part="SW1" gate="G$1" x="132.08" y="154.94" rot="R90"/>
-<instance part="TP1" gate="G$1" x="58.42" y="25.4"/>
 <instance part="R1" gate="G$1" x="10.16" y="157.48" smashed="yes" rot="R90">
 <attribute name="NAME" x="13.716" y="155.194" size="1.778" layer="95" font="vector" ratio="12" rot="R90"/>
 <attribute name="VALUE" x="16.002" y="155.194" size="1.778" layer="96" font="vector" ratio="12" rot="R90"/>
 </instance>
+<instance part="GND1" gate="1" x="210.82" y="116.84" smashed="yes" rot="MR0"/>
+<instance part="PWR2" gate="G$1" x="210.82" y="132.08" smashed="yes">
+<attribute name="VALUE" x="207.264" y="136.906" size="1.778" layer="96" font="vector" ratio="12"/>
+</instance>
+<instance part="CON2" gate="G$1" x="220.98" y="116.84"/>
+<instance part="TP1" gate="G$1" x="45.72" y="76.2"/>
+<instance part="TP2" gate="G$1" x="177.8" y="106.68" rot="R180"/>
+<instance part="TP5" gate="G$1" x="170.18" y="86.36" rot="R180"/>
 </instances>
 <busses>
@@
 <pinref part="GND57" gate="1" pin="GND"/>
 </segment>
+<segment>
+<pinref part="GND1" gate="1" pin="GND"/>
+<wire x1="215.9" y1="119.38" x2="210.82" y2="119.38" width="0.1524" layer="91"/>
+<wire x1="210.82" y1="119.38" x2="210.82" y2="116.84" width="0.1524" layer="91"/>
+<pinref part="CON2" gate="G$1" pin="GND@9"/>
+</segment>
 </net>
 <net name="TGT_TX" class="0">
@@
 <pinref part="IC3" gate="G$1" pin="VDD"/>
 <pinref part="PWR21" gate="G$1" pin="+3.3V_IF"/>
+</segment>
+<segment>
+<pinref part="PWR2" gate="G$1" pin="+3.3V_IF"/>
+<wire x1="215.9" y1="129.54" x2="210.82" y2="129.54" width="0.1524" layer="91"/>
+<wire x1="210.82" y1="129.54" x2="210.82" y2="132.08" width="0.1524" layer="91"/>
+<pinref part="CON2" gate="G$1" pin="VCC"/>
 </segment>
 </net>
@@
 <label x="71.12" y="121.92" size="1.778" layer="95" font="vector" ratio="12"/>
 </segment>
+<segment>
+<wire x1="248.92" y1="119.38" x2="256.54" y2="119.38" width="0.1524" layer="91"/>
+<label x="259.08" y="119.38" size="1.778" layer="95"/>
+<pinref part="CON2" gate="G$1" pin="NRESET"/>
+</segment>
 </net>
 <net name="IF_SWCLK" class="0">
 <segment>
 <pinref part="IC3" gate="G$1" pin="SWCLK/PIO0_10/SCK0/CT16B0_MAT2"/>
-<wire x1="76.2" y1="81.28" x2="45.72" y2="81.28" width="0.1524" layer="91"/>
+<wire x1="76.2" y1="81.28" x2="58.42" y2="81.28" width="0.1524" layer="91"/>
 <label x="48.26" y="81.28" size="1.778" layer="95" font="vector" ratio="12"/>
-<pinref part="TP12" gate="G$1" pin="TP"/>
+</segment>
+<segment>
+<wire x1="248.92" y1="127" x2="256.54" y2="127" width="0.1524" layer="91"/>
+<label x="259.08" y="127" size="1.778" layer="95"/>
+<pinref part="CON2" gate="G$1" pin="SWCLK"/>
 </segment>
 </net>
@@
 <segment>
 <pinref part="IC3" gate="G$1" pin="SWDIO/PIO0_15/AD4/CT32B1_MAT2"/>
-<wire x1="76.2" y1="68.58" x2="45.72" y2="68.58" width="0.1524" layer="91"/>
-<label x="53.34" y="68.58" size="1.778" layer="95" font="vector" ratio="12"/>
-<pinref part="TP11" gate="G$1" pin="TP"/>
+<wire x1="76.2" y1="68.58" x2="58.42" y2="68.58" width="0.1524" layer="91"/>
+<label x="48.26" y="68.58" size="1.778" layer="95" font="vector" ratio="12"/>
+</segment>
+<segment>
+<wire x1="248.92" y1="129.54" x2="256.54" y2="129.54" width="0.1524" layer="91"/>
+<label x="259.08" y="129.54" size="1.778" layer="95"/>
+<pinref part="CON2" gate="G$1" pin="SWDIO"/>
 </segment>
 </net>
@@
 <segment>
 <pinref part="IC3" gate="G$1" pin="PIO0_2/SSEL0/CT16B0_CAP0"/>
-<wire x1="76.2" y1="101.6" x2="71.12" y2="101.6" width="0.1524" layer="91"/>
+<wire x1="76.2" y1="101.6" x2="60.96" y2="101.6" width="0.1524" layer="91"/>
 <label x="48.26" y="101.6" size="1.778" layer="95" font="vector" ratio="12"/>
 </segment>
@@
 <segment>
 <pinref part="IC3" gate="G$1" pin="PIO0_1/CLKOUT/CT32B0_MAT2/USB_FTOGGLE"/>
-<wire x1="76.2" y1="104.14" x2="71.12" y2="104.14" width="0.1524" layer="91"/>
+<wire x1="76.2" y1="104.14" x2="58.42" y2="104.14" width="0.1524" layer="91"/>
 <label x="48.26" y="104.14" size="1.778" layer="95" font="vector" ratio="12"/>
 </segment>
@@
 <segment>
 <pinref part="IC3" gate="G$1" pin="PIO0_4/SCL"/>
-<wire x1="76.2" y1="96.52" x2="43.18" y2="96.52" width="0.1524" layer="91"/>
-<label x="33.02" y="96.52" size="1.778" layer="95" font="vector" ratio="12"/>
+<wire x1="76.2" y1="96.52" x2="58.42" y2="96.52" width="0.1524" layer="91"/>
+<label x="48.26" y="96.52" size="1.778" layer="95" font="vector" ratio="12"/>
 </segment>
 </net>
@@
 <segment>
 <pinref part="IC3" gate="G$1" pin="PIO0_5/SDA"/>
-<wire x1="76.2" y1="93.98" x2="43.18" y2="93.98" width="0.1524" layer="91"/>
-<label x="33.02" y="93.98" size="1.778" layer="95" font="vector" ratio="12"/>
+<wire x1="76.2" y1="93.98" x2="58.42" y2="93.98" width="0.1524" layer="91"/>
+<label x="48.26" y="93.98" size="1.778" layer="95" font="vector" ratio="12"/>
 </segment>
 </net>
@@
 <segment>
 <pinref part="CON14" gate="G$1" pin="VCC"/>
-<wire x1="81.28" y1="25.4" x2="58.42" y2="25.4" width="0.1524" layer="91"/>
+<wire x1="81.28" y1="25.4" x2="66.04" y2="25.4" width="0.1524" layer="91"/>
 <label x="60.96" y="25.4" size="1.778" layer="95" font="vector" ratio="12"/>
-<pinref part="TP1" gate="G$1" pin="TP"/>
 </segment>
 </net>
@@
 <wire x1="76.2" y1="71.12" x2="45.72" y2="71.12" width="0.1524" layer="91"/>
 <pinref part="TP13" gate="G$1" pin="TP"/>
-<label x="53.34" y="71.12" size="1.778" layer="95" font="vector" ratio="12"/>
-</segment>
-</net>
+<label x="48.26" y="71.12" size="1.778" layer="95" font="vector" ratio="12"/>
+</segment>
+</net>
+<net name="N$1" class="0">
+<segment>
+<pinref part="TP1" gate="G$1" pin="TP"/>
+<pinref part="IC3" gate="G$1" pin="TMS/PIO0_12/AD1/CT32B1_CAP0"/>
+<wire x1="45.72" y1="76.2" x2="76.2" y2="76.2" width="0.1524" layer="91"/>
+</segment>
+</net>
+<net name="N$5" class="0">
+<segment>
+<pinref part="IC3" gate="G$1" pin="PIO0_16/AD5/CT32B1_MAT3/WAKEUP"/>
+<pinref part="TP2" gate="G$1" pin="TP"/>
+<wire x1="177.8" y1="106.68" x2="170.18" y2="106.68" width="0.1524" layer="91"/>
+</segment>
+</net>
+<net name="N$6" class="0">
+<segment>
+<pinref part="IC3" gate="G$1" pin="PIO1_15/!DCD!/CT16B0_MAT2/SCK1"/>
+<pinref part="TP5" gate="G$1" pin="TP"/>
+</segment>
+</net>

Commit message: Refactor of repository
Parts:
- removed C15: 18pF, mbed-HDK:C0603
- removed CON14: SWD-10/TC2050_SMD, mbed-HDK-Connector:SWD-10/TC2050_SMD
- removed R13: 470R, mbed-HDK:R0603
- removed R18: 33R, mbed-HDK:R0603
- added C2: 10uF, mbed-HDK:C0603
- added CON3: SWD-10/TC2050_SMD, mbed-HDK-Connector:SWD-10/TC2050_SMD
- added R2: 470R, mbed-HDK:R0603
- added R4: 0R@DNF, mbed-HDK:R0402
- C1: value 10uF -> 100nF
- C6: value 100nF -> 18pF
- D1: device mbed-HDK:BAT60A -> mbed-HDK-Transistor:BAT60J
- R1: value 0R@DNF -> 470R; device mbed-HDK:R0402 -> mbed-HDK:R0603
- R11: value 470R -> 33R
- renumbered C12 to C4, C16 to C7, C17 to C9, C18 to C8, C19 to C3, C20 to C5, CON9 to CON1, LED4 to LED3, LED5 to LED1, LED6 to LED2, R12 to R3, R15 to R6, R16 to R5, R17 to R10, R19 to R9, R20 to R7, R21 to R8
Connections:
- net +3.3V_IF: now also C2.P$1, CON3.VCC, R1.P$1, R2.P$1; no longer C6.P$1, CON2.VCC, R11.P$1, R13.P$1
- net GND: now also C2.P$2, CON2.GND@3, CON2.GND@5, CON3.GND@9; no longer C15.P$2, CON14.GND@3, CON14.GND@5, CON14.GND@9
- net IF_NRESET: now also CON3.NRESET; no longer CON2.NRESET
- net IF_SWCLK: now also CON3.SWCLK; no longer CON2.SWCLK
- net IF_SWDIO: now also CON3.SWDIO; no longer CON2.SWDIO
- net N$18: now also C6.P$1; no longer C15.P$1
- net N$2: now also R2.P$2; no longer R11.P$2
- net N$7: now also R1.P$2; no longer R13.P$2
- net TGT_NRESET: now also CON2.NRESET; no longer CON14.NRESET
- net TGT_RTS: now also R4.P$2; no longer R1.P$2
- net TGT_RX: now also CON2.TGT_RX; no longer CON14.TGT_RX
- net TGT_SWCLK: now also CON2.SWCLK, R4.P$1; no longer CON14.SWCLK, R1.P$1
- net TGT_SWDIO: now also CON2.SWDIO; no longer CON14.SWDIO
- net TGT_TX: now also CON2.TGT_TX; no longer CON14.TGT_TX
- net USB-D+: now also R11.P$1; no longer R18.P$1
- net USB_DP: now also R11.P$2; no longer R18.P$2
- net V_ISENSE: now also CON2.VCC; no longer CON14.VCC
